File: SuperHAT V2.kicad_pcb (KiCad board)
At the start: 4 copper layers, 65 x 56.5 mm, 66 parts, among them J1 GPIO, J10 Qwiic_RA, J11 BM02B-GHS-TBT_LF__SN_, J13 SM02B-PASS-TBTLFSN, J2 Conn_01x03, J4 Conn_01x03, J5 Qwiic_RA, J6 Qwiic_Vertical, J7 Qwiic_Vertical, J8 SM04B-GHS-TB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

Commit message: No errors before generating BOM.
Connections:
- U2 pad 7: Net-(U2-GND-Pad7) -> GND
- U2 pad 9: Net-(U2-GND-Pad7) -> GND
Routing:
- net Net-(U2-GND-Pad7): vias 1 -> 0
- net GND: vias 35 -> 36
