File: SuperHAT V2.kicad_sch (KiCad schematic)
At the start: 64 parts, among them J1 GPIO, J10 Qwiic_RA, J11 BM02B-GHS-TBT_LF__SN_, J13 SM02B-PASS-TBTLFSN, J2 Conn_01x03, J4 Conn_01x03, J5 Qwiic_RA, J6 Qwiic_Vertical, J7 Qwiic_Vertical, J8 SM04B-GHS-TB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

Commit message: Committing before creating HTML BOM, in case if it messes things up.
Parts:
- J1: Mfr. # 2187 -> (none); Mfr. Part # (none) -> 2187
- J11: Availability In Stock -> (none); Check_prices https://www.snapeda.com/parts/BM02B-GHS-TBT(LF)(SN)/JST/vie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 -> (none); Description_1 Connector Header Surface Mount 2 position 0.049 (1.25mm) -> (none); MANUFACTURER JST Sales -> (none); MAXIMUM_PACKAGE_HEIGHT 4.05 mm -> (none); Mfr. # BM02B-GHS-TBT(LF)(SN) -> (none); Mfr. Part # (none) -> BM02B-GHS-TBT(LF)(SN); Order Link (none) -> https://www.digikey.com/en/products/detail/jst-sales-americ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; PARTREV NA -> (none); Package None -> (none); Price None -> $0.33; Purchase-URL https://www.snapeda.com/api/url_track_click_mouser/?unipart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 -> (none); STANDARD Manufacturer Recommendations -> (none); SnapEDA_Link https://www.snapeda.com/parts/BM02B-GHS-TBT(LF)(SN)/JST/vie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 -> (none)
- J13: Mfr. # SM02B-PASS-TBT -> (none); Mfr. Part # (none) -> SM02B-PASS-TBT
- J3: Mfr. # MR30PW-M -> (none); Mfr. Part # (none) -> MR30PW-M
- JP5: Availability In Stock -> (none); Check_prices https://www.snapeda.com/parts/B04B-PASK-1/JST+Sales+America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 -> (none); Description_1 Connector Header Through Hole 4 position 0.079 (2.00mm) -> (none); Mfr. # B04B-PASK-1 -> (none); Mfr. Part # (none) -> B04B-PASK-1; SnapEDA_Link https://www.snapeda.com/parts/B04B-PASK-1/JST+Sales+America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 -> (none)
- R1: Mfr. # CHP0805AFX-1001ELF -> (none); Mfr. Part # (none) -> CHP0805AFX-1001ELF
- R10: Mfr. # WSLP0805R0400DEA -> (none); Mfr. Part # (none) -> WSLP0805R0400DEA
- R16: Mfr. # WSLP0805R1000FEA -> (none); Mfr. Part # (none) -> WSLP0805R1000FEA
- R2: Mfr. # CMP0805AFX-3300ELF -> (none); Mfr. Part # (none) -> CMP0805AFX-3300ELF
- R7: Mfr. # SG73S2ATTD3002F -> (none); Mfr. Part # (none) -> SG73S2ATTD3002F
- R8: Mfr. # CMP0805AFX-1004ELF -> (none); Mfr. Part # (none) -> CMP0805AFX-1004ELF
- RN3: Mfr. # EXB-2HV103JV -> (none); Mfr. Part # (none) -> EXB-2HV103JV
- RV1: Mfr. # TC33X-1-103ETC33X-1-103E -> (none); Mfr. Part # (none) -> TC33X-1-103ETC33X-1-103E
- U1: Mfr. # INA3221AQRGVRQ1 -> (none); Mfr. Part # (none) -> INA3221AQRGVRQ1
- U2: Mfr. # DRV8871DDARQ1 -> (none); Mfr. Part # (none) -> DRV8871DDARQ1
- U3: Mfr. # DRV8825PWPR -> (none); Mfr. Part # (none) -> DRV8825PWPR

Commit message: Beautiful BOM.
Parts:
- C3: Mfr. # C0805C103K5TACAUTO -> (none); Mfr. Part # (none) -> C0805C103K5TACAUTO
- C4: Mfr. # C0805C474J9RACTU -> (none); Mfr. Part # (none) -> C0805C474J9RACTU
- D14: Mfr. # GSD2004WS-HE3-08 -> (none); Mfr. Part # (none) -> GSD2004WS-HE3-08
- J10: Mfr. # SM04B-SRSS-TB -> (none); Mfr. Part # (none) -> SM04B-SRSS-TB
- J2, J4: Mfr. (none) -> Würth Elektronik; Mfr. Part # (none) -> 61300311121; Order Link https://www.amazon.com/Straight-Breakaway-Connector-Breadbo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 -> https://www.digikey.com/en/products/detail/w%C3%BCrth-elekt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; Price $0.00 -> $0.12
Changed lines of the file:
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@@
 			)
 		)
-		(property "Mfr. #" "SM04B-SRSS-TB"
+		(property "Mfr. Part #" "SM04B-SRSS-TB"
 			(at 254 63.5 0)
 			(effects
@@
 			)
 		)
-		(property "Mfr. Part #" ""
-			(at 254 53.34 0)
-			(effects
-				(font
-					(size 1.27 1.27)
-				)
-				(hide yes)
-			)
-		)
-		(property "PROD_ID" ""
-			(at 254 53.34 0)
-			(effects
-				(font
-					(size 1.27 1.27)
-				)
-				(hide yes)
-			)
-		)
-		(property "Sim.Device" ""
-			(at 254 53.34 0)
-			(effects
-				(font
-					(size 1.27 1.27)
-				)
-				(hide yes)
-			)
-		)
-		(property "Sim.Pins" ""
-			(at 254 53.34 0)
-			(effects
-				(font
-					(size 1.27 1.27)
-				)
-				(hide yes)
-			)
-		)
-		(property "Sim.Type" ""
-			(at 254 53.34 0)
-			(effects
-				(font
-					(size 1.27 1.27)
-				)
-				(hide yes)
-			)
-		)
-		(property "MF" ""
-			(at 254 53.34 0)
-			(effects
-				(font
-					(size 1.27 1.27)
-				)
-				(hide yes)
-			)
-		)
-		(property "MP" ""
-			(at 254 53.34 0)
-			(effects
-				(font
-					(size 1.27 1.27)
-				)
-				(hide yes)
-			)
-		)
-		(property "REFERENCE" ""
-			(at 254 53.34 0)
-			(effects
-				(font
-					(size 1.27 1.27)
-				)
-				(hide yes)
-			)
-		)
 		(pin "4"
 		)
@@
 			)
 		)
-		(property "Mfr. #" "C0805C103K5TACAUTO"
+		(property "Mfr. Part #" "C0805C103K5TACAUTO"
 			(at 168.91 135.89 90)
 			(effects
@@
 			)
 		)
-		(property "Mfr. #" "C0805C474J9RACTU"
+		(property "Mfr. Part #" "C0805C474J9RACTU"
 			(at 194.31 129.54 90)
 			(effects
@@
 			)
 		)
-		(property "Mfr. #" "GSD2004WS-HE3-08"
+		(property "Mfr. Part #" "GSD2004WS-HE3-08"
 			(at 106.68 99.06 0)
 			(effects
@@
 			)
 		)
-		(property "Datasheet" "~"
+		(property "Datasheet" "https://www.we-online.com/components/products/datasheet/61300311121.pdf"
 			(at 238.76 133.35 0)
 			(effects
@@
 			)
 		)
-		(property "Mfr." ""
+		(property "Mfr." "Würth Elektronik"
 			(at 238.76 124.46 0)
 			(effects
@@
 			)
 		)
-		(property "Mfr. Part #" ""
+		(property "Mfr. Part #" "61300311121"
 			(at 238.76 124.46 0)
 			(effects
@@
 			)
 		)
-		(property "Price" "$0.00"
+		(property "Price" "$0.12"
 			(at 238.76 124.46 0)
 			(effects
@@
 			)
 		)
-		(property "Order Link" "https://www.amazon.com/Straight-Breakaway-Connector-Breadboard-Electronic/dp/B09MYBRW3F?crid=3JR0BZNCU8K8J&dib=eyJ2IjoiMSJ9.3vFjmsH10W3-0I49M7i2SLer6N2w76n3suAL41lNyWbCktqeX2xUwJKGOw1Unq-mAp24IQL2WQ-Ev7Umi65YUYWwukLOeoqjLE4MCKmsExRo7y7O8beFGF-NY-mrllV9VKK4tI6JlMWT6oqZ_rCOCrXUoStfaWefHyDqNKRyilyns3IozKEM_18D3NupDy3bF_TYgvEPFbIX5EQWrNKwcTDbRlgYyJ1qEApCaPAYdds.HCWtlvjyp8dekPH4j2M5xTF1mJrDF1h5rp-JmzUzVHE&dib_tag=se&keywords=male%2Bpin%2Bheaders&qid=1735364673&sprefix=male%2Bpin%2Bheaders%2Caps%2C130&sr=8-8&th=1"
+		(property "Order Link" "https://www.digikey.com/en/products/detail/w%C3%BCrth-elektronik/61300311121/4846825"
 			(at 238.76 124.46 0)
 			(effects
@@
 			)
 		)
-		(property "Datasheet" "~"
+		(property "Datasheet" "https://www.we-online.com/components/products/datasheet/61300311121.pdf"
 			(at 238.76 121.92 0)
 			(effects
@@
 			)
 		)
-		(property "Mfr." ""
+		(property "Mfr." "Würth Elektronik"
 			(at 238.76 113.03 0)
 			(effects
@@
 			)
 		)
-		(property "Mfr. Part #" ""
+		(property "Mfr. Part #" "61300311121"
 			(at 238.76 113.03 0)
 			(effects
@@
 			)
 		)
-		(property "Price" "$0.00"
+		(property "Price" "$0.12"
 			(at 238.76 113.03 0)
 			(effects
@@
 			)
 		)
-		(property "Order Link" "https://www.amazon.com/Straight-Breakaway-Connector-Breadboard-Electronic/dp/B09MYBRW3F?crid=3JR0BZNCU8K8J&dib=eyJ2IjoiMSJ9.3vFjmsH10W3-0I49M7i2SLer6N2w76n3suAL41lNyWbCktqeX2xUwJKGOw1Unq-mAp24IQL2WQ-Ev7Umi65YUYWwukLOeoqjLE4MCKmsExRo7y7O8beFGF-NY-mrllV9VKK4tI6JlMWT6oqZ_rCOCrXUoStfaWefHyDqNKRyilyns3IozKEM_18D3NupDy3bF_TYgvEPFbIX5EQWrNKwcTDbRlgYyJ1qEApCaPAYdds.HCWtlvjyp8dekPH4j2M5xTF1mJrDF1h5rp-JmzUzVHE&dib_tag=se&keywords=male%2Bpin%2Bheaders&qid=1735364673&sprefix=male%2Bpin%2Bheaders%2Caps%2C130&sr=8-8&th=1"
+		(property "Order Link" "https://www.digikey.com/en/products/detail/w%C3%BCrth-elektronik/61300311121/4846825"
 			(at 238.76 113.03 0)
 			(effects

Commit message: Schematic changes made.
Parts:
- removed RN3: 10k, 10k Resistor Array:RES_EXB2HV, symbol Device:R_Pack08
- added R12: 10k, 0805 Resistor Moisture Resistant:RES_CHP0805_BRN, symbol Device:R
- added RN1, RN2, RN4, RN5: 10k, 2 RES 10k Array:SMT_1002P1AT_VIS, symbol Device:R_Pack02
Connections:
- net +3V3: now also RN1.2 (R2.1), RN2.3 (R2.2), RN4.2 (R2.1)
- net GND: now also R12.2, RN1.1 (R1.1), RN2.4 (R1.2), RN4.1 (R1.1), RN5.4 (R1.2)
- net GPIO11/SPI0.SCLK: now also Q2.1 (G), R4.1, RN2.1 (R1.1)
- net GPIO14/TXD0: no longer Q3.1 (G), R5.1
- net GPIO15/RXD0: no longer Q1.1 (G), R3.1
- net GPIO16: now also RN5.1 (R1.1)
- net GPIO17: now also Q1.1 (G), R3.1, RN1.4 (R1.2)
- net GPIO18/PCM.CLK: now also Q3.1 (G), R5.1, RN4.4 (R1.2)
- net GPIO6: no longer Q2.1 (G), R4.1
- net PV: now reaches U1.10 (PV)
- net PV: now also RN5.3 (R2.2)
- net VPU: now reaches U1.16 (VPU)
- net VPU: now also RN5.2 (R2.1)
- net CRITICAL: now reaches U1.9 (CRITICAL)
- net CRITICAL: now also RN4.3 (R2.2)
- net WARNING: now reaches U1.8 (WARNING)
- net WARNING: now also RN1.3 (R2.2)
- net TC: now reaches U1.13 (TC)
- net TC: now also RN2.2 (R2.1)
- net at U1.5 (A0): now also R12.1
Other:
- moved on the sheet: J11, J2, J4

Commit message: Fixed MOSFET circuits, pin values, and diode layout.
Parts:
- removed U2: DRV8871DDA, Package_SO:Texas_HTSOP-8-1EP_3.9x4.9mm_P1.27mm_EP2.95x4.9mm_Mask2.4x3.1mm_ThermalVias, symbol Driver_Motor:DRV8871DDA
- added JP10, JP7, JP8, JP9: SolderJumper_2_Open, Jumper:SolderJumper-2_P1.3mm_Open_TrianglePad1.0x1.5mm, symbol Jumper:SolderJumper_2_Open
- added U4: DRV8871DDA, Package_SO:Texas_HTSOP-8-1EP_3.9x4.9mm_P1.27mm_EP2.95x4.9mm_Mask2.4x3.1mm_ThermalVias, symbol Driver_Motor:DRV8871DDA
Connections:
- net +12V: now also U4.5 (VM)
- net +3V3: now also RN2.2 (R2.1), RN4.1 (R1.1); no longer RN2.3 (R2.2), RN4.2 (R2.1)
- net CRITICAL: now also RN4.4 (R1.2); no longer RN4.3 (R2.2)
- net GND: now also RN1.4 (R1.2), RN4.3 (R2.2), RN5.2 (R2.1), U4.1 (GND), U4.7 (GND), U4.9 (GND); no longer RN1.1 (R1.1), RN4.1 (R1.1), RN5.4 (R1.2)
- net GPIO10/SPI0.MOSI: now also U4.2 (IN2)
- net GPIO16: now also RN5.3 (R2.2); no longer RN5.1 (R1.1)
- net GPIO17: now also RN1.1 (R1.1); no longer RN1.4 (R1.2)
- net GPIO18/PCM.CLK: now also RN4.2 (R2.1); no longer RN4.4 (R1.2)
- net GPIO9/SPI0.MISO: now also U4.3 (IN1)
- net PV: now also RN5.1 (R1.1); no longer RN5.3 (R2.2)
- net TC: now also RN2.3 (R2.2); no longer RN2.2 (R2.1)
- net VPU: now also RN5.4 (R1.2); no longer RN5.2 (R2.1)
- net at D12.A, JP4.1, Q4.3 (D): now also JP10.1 (A); no longer D14.A
- net at D2.A, JP1.1, Q1.3 (D): now also JP7.1 (A); no longer D3.A
- net at D6.A, JP2.1, Q2.3 (D): now also JP8.1 (A); no longer D8.A
- net at R7.1: now also U4.4 (ILIM)
- net at D9.A, JP3.1, Q3.3 (D): now also JP9.1 (A); no longer D11.A
- net at J13.1: now also U4.6 (OUT1)
- net at J13.2: now also U4.8 (OUT2)
- new net: D8.A, JP8.2 (B)
- new net: D11.A, JP9.2 (B)
- new net: D3.A, JP7.2 (B)
- new net: D14.A, JP10.2 (B)
Other:
- moved on the sheet: RN4, RN5

Commit message: Added overvoltage protection to schematic.
Parts:
- added C11: 10 nF, symbol Device:C_Small
- added R13: 10k, 0805 Resistor Moisture Resistant:RES_CHP0805_BRN, symbol Device:R
- added R14: 453, symbol Device:R
- added R17: 400k, symbol Device:R
- added R18: 7.5k, symbol Device:R
- added R19: 2.4k, symbol Device:R
- added U2: TPS259631DDAR, TPS259631:SOIC_20DDAR_TEX, symbol TPS259631:TPS259620DDAR
- R3, R4, R5, R6: value 33 -> 100; footprint CMP0805AFX:RES_CMP0805_BRN -> 0805 Resistor Moisture Resistant:RES_CHP0805_BRN; Mfr. Part # CMP0805AFX-33R0ELF -> CHP0805AFX-1000ELF; Order Link https://www.digikey.com/en/products/detail/bourns-inc/CMP08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 -> https://www.digikey.com/en/products/detail/bourns-inc/CHP08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; Price $0.26 -> $0.38
Connections:
- net +3V3: now also R13.2
- net +5V: now also R18.2, U2.4 (IN); no longer J1.2 (Pin_2), J1.4 (Pin_4), J10.2 (Pin_2)
- net GND: now also C11.1, R14.2, R17.2, R19.2, U2.1 (GND), U2.9 (EPAD)
- net GPIO27: now also R13.1, U2.6 (*FLT)
- new net: R18.1, R19.1, U2.3 (EN/UVLO)
- new net: C11.2, U2.2 (DVDT)
- new net: R14.1, U2.7 (ILM)
- new net: R17.1, U2.8 (OVCSEL)
- new net +5VPI: J1.2 (Pin_2), J1.4 (Pin_4), J10.2 (Pin_2), U2.5 (OUT)
Other:
- moved on the sheet: JP10, JP8, JP9

Commit message: Overvoltage protection laid out on footprint.
Parts:
- removed J11: BM02B-GHS-TBT_LF__SN_, BM02B-GHS-TBT:BM02B-GHS-TBT, symbol BM02B-GHS-TBT:BM02B-GHS-TBT_LF__SN_
- removed J13: SM02B-PASS-TBTLFSN, SM02B-PASS-TBT:CONN_SM02B-PASS_JST, symbol SM02B-PASS-TBT:SM02B-PASS-TBTLFSN
- added C12: 0.1 uF, 0805 Ceramic Capacitor:CAPC2012X140N, symbol Device:C_Small
- added J11: Conn_01x02, Connector_PinHeader_2.54mm:PinHeader_1x02_P2.54mm_Horizontal, symbol Connector_Generic:Conn_01x02
- added J12: B02B-PASK-1, B02B-PASK-1:CONN_B02B-PASK-1_JST, symbol B02B-PASK-1:B02B-PASK-1
- C11: footprint (none) -> 0805 Ceramic Capacitor:CAPC2012X140N; Mfr.  (none) -> KEMET; Mfr. Part # (none) -> C0805C103K5TACAUTO; Order Link (none) -> https://www.digikey.com/en/products/detail/kemet/C0805C103K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; Price (none) -> $0.553
- J10, J5: PROD_ID (none) -> CONN-13694
- R12, R13: Mfr. (none) -> Bourns Inc.; Mfr. Part # (none) -> CHP0805AFX-1002ELF; Order Link (none) -> https://www.digikey.com/en/products/detail/bourns-inc/CHP08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; Price (none) -> $0.38
- R14: footprint (none) -> RESC2012X60N:RESC2012X60N; Mfr. (none) -> KOA Speer Electronics, Inc.; Mfr. Part # (none) -> RN73R2ATTD4530B25; Order Link (none) -> https://www.digikey.com/en/products/detail/koa-speer-electr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; Price (none) -> $0.23
- R17: value 400k -> 470k; footprint (none) -> CMP0805AFX:RES_CMP0805_BRN; Mfr. (none) -> Bourns Inc.; Mfr. Part # (none) -> CMP0805AFX-4703ELF; Order Link (none) -> https://www.digikey.com/en/products/detail/bourns-inc/CMP08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; Price (none) -> $0.23
- R18: footprint (none) -> TNPW0805:RES_TNPW0805_VIS; Mfr. (none) -> Vishay Dale; Mfr. Part # (none) -> TNPW08057K50BEEA; Order Link (none) -> https://www.digikey.com/en/products/detail/vishay-dale/TNPW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; Price (none) -> $0.39
- R19: footprint (none) -> TNPW0805:RES_TNPW0805_VIS
- U2: Mfr. (none) -> Texas Instruments; Mfr. Part # (none) -> TPS259621DDAR; Order Link (none) -> https://www.digikey.com/en/products/detail/texas-instrument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; Price (none) -> $0.81
Connections:
- net +3V3: now also R13.1; no longer R13.2
- net +5V: now also R18.1, J11.2 (Pin_2); no longer R18.2
- net +5VPI: now also C12.2
- net GND: now also C11.2, C12.1, J11.1 (Pin_1); no longer C11.1
- net GPIO27: now also R13.2; no longer R13.1
- net at U4.6 (OUT1): now also J12.2
- net at U4.8 (OUT2): now also J12.1
- net at R19.1, U2.3 (EN/UVLO): now also R18.2; no longer R18.1
- net at U2.2 (DVDT): now also C11.1; no longer C11.2

Commit message: Pre footprint migration to create BOM V2
Parts:
- C1, C10, C12, C5, C6, C7, C8: Mfr. Part # C0805C104J5RACAUTO -> (none); Part # (none) -> C0805C104J5RACAUTO
- C11, C3: Mfr. Part # C0805C103K5TACAUTO -> (none); Part # (none) -> C0805C103K5TACAUTO
- C2, C9: Mfr. Part # T598D476M025ATE060 -> (none); Part # (none) -> T598D476M025ATE060
- C4: Mfr. Part # C0805C474J9RACTU -> (none); Part # (none) -> C0805C474J9RACTU
- D1, D10, D13, D7: Mfr. Part # 150080GS75000 -> (none); Part # (none) -> 150080GS75000
- D11, D12, D14, D2, D3, D6, D8, D9: Mfr. Part # GSD2004WS-HE3-08 -> (none); Part # (none) -> GSD2004WS-HE3-08
- D4, D5: Mfr. Part # 150080RS75000 -> (none); Part # (none) -> 150080RS75000
- J1: Mfr. Adafruit -> SparkFun; Mfr. Part # 2187 -> (none); Order Link https://www.adafruit.com/product/2187 -> https://www.digikey.com/en/products/detail/sparkfun-electro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; Part # (none) -> PRT-14017; Price $1.95 -> $2.75
- J10, J5: Mfr. Part # SM04B-SRSS-TB -> (none); PROD_ID CONN-13694 -> (none); Part # (none) -> SM04B-SRSS-TB
- J11: Mfr. Part # 10129379-902002BLF -> (none); Part # (none) -> 10129379-902002BLF
- J12: Mfr. (none) -> JST Sales America Inc.; Order Link (none) -> https://www.digikey.com/en/products/detail/jst-sales-americ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; Part # (none) -> B02B-PASK-1; Price (none) -> $0.16
- J2, J4: Mfr. Part # 61300311121 -> (none); Part # (none) -> 61300311121
- J3: Mfr. Part # MR30PW-M -> (none); Part # (none) -> MR30PW-M
- J6, J7: Mfr. Part # BM04B-SRSS-TB -> (none); Part # (none) -> BM04B-SRSS-TB
- J8, J9: Mfr. Part # SM04B-GHS-TB -> (none); Part # (none) -> SM04B-GHS-TB
- JP1, JP3: Mfr. Part # B03B-PASK-1 -> (none); Part # (none) -> B03B-PASK-1
- JP5: Mfr. Part # B04B-PASK-1 -> (none); Part # (none) -> B04B-PASK-1
- Q1, Q2, Q3, Q4: Mfr. Part # AOSS32136C -> (none); Part # (none) -> AOSS32136C
- R1: value 1k -> 3k; footprint 0805 Resistor Moisture Resistant:RES_CHP0805_BRN -> TNPW0805:RES_TNPW0805_VIS; Mfr. Bourns Inc. -> Vishay Dale; Mfr. Part # CHP0805AFX-1001ELF -> (none); Order Link https://www.digikey.com/en/products/detail/bourns-inc/CHP08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 -> https://www.digikey.com/en/products/detail/vishay-dale/TNPW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; Part # (none) -> TNPW08053K00BEEA; Price $0.46 -> $0.39
- R10, R11, R9: Mfr. Part # WSLP0805R0400DEA -> (none); Part # (none) -> WSLP0805R0400DEA
- R12, R13: Mfr. Part # CHP0805AFX-1002ELF -> (none); Part # (none) -> CHP0805AFX-1002ELF
- R14: Mfr. Part # RN73R2ATTD4530B25 -> (none); Part # (none) -> RN73R2ATTD4530B25
- R15, R16: Mfr. Part # WSLP0805R1000FEA -> (none); Part # (none) -> WSLP0805R1000FEA
- R17: Mfr. Part # CMP0805AFX-4703ELF -> (none); Part # (none) -> CMP0805AFX-4703ELF
- R18: Mfr. Part # TNPW08057K50BEEA -> (none); Part # (none) -> TNPW08057K50BEEA
- R19: Mfr. (none) -> Vishay Dale; Order Link (none) -> https://www.digikey.com/en/products/detail/vishay-dale/TNPW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; Part # (none) -> TNPW08052K40BEEA; Price (none) -> $0.39
- R2: value 330 -> 1k; footprint 0805 330 Ohm Resistor Moisture Resistant:RES_CMP0805_BRN -> TNPW0805:RES_TNPW0805_VIS; Mfr. (none) -> Vishay Dale; Mfr.  Bourns Inc. -> (none); Mfr. Part # CMP0805AFX-3300ELF -> (none); Order Link https://www.digikey.com/en/products/detail/bourns-inc/CMP08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 -> https://www.digikey.com/en/products/detail/vishay-dale/TNPW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; Part # (none) -> TNPW08051K00BEEA; Price $0.26 -> $0.39
- R3, R4, R5, R6: Mfr. Part # CHP0805AFX-1000ELF -> (none); Part # (none) -> CHP0805AFX-1000ELF
- R7: Mfr. Part # SG73S2ATTD3002F -> (none); Part # (none) -> SG73S2ATTD3002F
- R8: Mfr. Part # CMP0805AFX-1004ELF -> (none); Part # (none) -> CMP0805AFX-1004ELF
- RN1, RN2, RN5: Mfr. (none) -> Vishay Beyschlag/Draloric/BC Components; Order Link (none) -> https://www.digikey.com/en/products/detail/vishay-beyschlag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; Part # (none) -> ACASN1002S1002P1AT; Price (none) -> $0.469
- RN4: Mfr.  (none) -> Vishay Beyschlag/Draloric/BC Components; Order Link (none) -> https://www.digikey.com/en/products/detail/vishay-beyschlag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; Part # (none) -> ACASN1002S1002P1AT; Price (none) -> $0.469
- RV1: Mfr. Part # TC33X-1-103ETC33X-1-103E -> (none); Part # (none) -> TC33X-1-103ETC33X-1-103E
- U1: Mfr. Part # INA3221AQRGVRQ1 -> (none); Part # (none) -> INA3221AQRGVRQ1
- U2: Mfr. Part # TPS259621DDAR -> (none); Part # (none) -> TPS259621DDAR
- U3: Mfr. Part # DRV8825PWPR -> (none); Part # (none) -> DRV8825PWPR
- U4: Mfr. (none) -> Texas Instruments; Order Link (none) -> https://www.digikey.com/en/products/detail/texas-instrument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; Part # (none) -> DRV8871DDARQ1; Price (none) -> $3.03
Connections:
- net GPIO20/PCM.DIN: no longer U3.20 (DIR)
- net GPIO26: now also U3.20 (DIR)
- net at U3.5 (AOUT1): now also JP5.1; no longer JP5.4
- net at U3.8 (BOUT2): now also JP5.4; no longer JP5.1
Other:
- moved on the sheet: C11, C12, R13, R14, R17, R18, R19, U2

Commit message: Bom acting goofy but I still generated one.
Parts:
- JP2, JP4: Mfr. Part # B03B-PASK-1 -> (none); Part # (none) -> B03B-PASK-1
Changed lines of the file:
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@@
 			)
 		)
-		(property "Mfr. Part #" "B03B-PASK-1"
+		(property "Part #" "B03B-PASK-1"
 			(at 77.47 99.06 0)
 			(effects
@@
 			)
 		)
-		(property "Mfr. Part #" "B03B-PASK-1"
+		(property "Part #" "B03B-PASK-1"
 			(at 25.4 154.94 0)
 			(effects
