File: SuperHAT V2.kicad_sch (KiCad schematic)
At the start: 80 parts, among them J1 GPIO, J10 Qwiic_RA, J11 Conn_01x02, J12 B02B-PASK-1, J2 Conn_01x03, J4 Conn_01x03, J5 Qwiic_RA, J6 Qwiic_Vertical, J7 Qwiic_Vertical, J8 SM04B-GHS-TB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

Commit message: SuperHAT V2
Parts:
- R19: value 2.4k -> 2.61k; Order Link https://www.digikey.com/en/products/detail/vishay-dale/TNPW08052K40BEEA/1607323 -> https://www.digikey.com/en/products/detail/vishay-dale/TNPW08052K61BEEN/1610534?s=N4IgjCBcoEwAwA4CsVQGMoDMCGAbAzgKYA0IA9lANogwB0AbGAAQDWA8gBYC2%2BIAuqQAOAFyggAqgDsAlsLaYAsoWz4ArgCdCIAL6kAtDFQgMkYetUlyVECj7bdNawBUAcgAUA6oji3tQA; Part # TNPW08052K40BEEA -> TNPW08052K61BEEN; Price $0.39 -> $0.67
- U2: value TPS259631DDAR -> TPS259621DDAR
Changed lines of the file:
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@@
 			)
 		)
-		(property "Value" "2.4k"
+		(property "Value" "2.61k"
 			(at -73.66 70.866 90)
 			(effects
@@
 			)
 		)
-		(property "Description" "RES 2.4K OHM 0.1% 0.26W 0805"
+		(property "Description" "RES 2.61K OHM 0.1% 0.26W 0805"
 			(at -73.66 64.77 0)
 			(effects
@@
 			)
 		)
-		(property "Part #" "TNPW08052K40BEEA"
+		(property "Part #" "TNPW08052K61BEEN"
 			(at -73.66 64.77 90)
 			(effects
@@
 			)
 		)
-		(property "Order Link" "https://www.digikey.com/en/products/detail/vishay-dale/TNPW08052K40BEEA/1607323"
+		(property "Order Link" "https://www.digikey.com/en/products/detail/vishay-dale/TNPW08052K61BEEN/1610534?s=N4IgjCBcoEwAwA4CsVQGMoDMCGAbAzgKYA0IA9lANogwB0AbGAAQDWA8gBYC2%2BIAuqQAOAFyggAqgDsAlsLaYAsoWz4ArgCdCIAL6kAtDFQgMkYetUlyVECj7bdNawBUAcgAUA6oji3tQA"
 			(at -73.66 64.77 90)
 			(effects
@@
 			)
 		)
-		(property "Price" "$0.39"
+		(property "Price" "$0.67"
 			(at -73.66 64.77 90)
 			(effects
@@
 			)
 		)
-		(property "Value" "TPS259631DDAR"
+		(property "Value" "TPS259621DDAR"
 			(at -57.4959 26.67 0)
 			(effects
